File: src/boards/ST2402/ST2402.kicad_sch (KiCad schematic)
At the start: 18 parts, among them J1 Conn_02x19_Odd_Even, J2 Conn_02x19_Odd_Even, J3 Conn_01x08, J4 Conn_01x08, J5 Conn_01x06, J6 Conn_01x10, J7 Conn_01x02, J8 Conn_01x02

Commit message: Added Mouser part numbers
Updated BOM and schematic with Mouser part numbers
Parts:
- J1, J2: Mouser ordercode (none) -> 200-SSQ11901GD
- J3, J4: Mouser ordercode (none) -> 200-SSQ10802GS
- J5: Mouser ordercode (none) -> 200-SSQ10602GS
- J6: Mouser ordercode (none) -> 200-SSQ11023GS
- J7, J8: Mouser ordercode (none) -> 200-SSQ10202GS
- TP4: value TestPoint -> YEL; Mouser ordercode (none) -> 534-5012
- TP5: value TestPoint -> ORG; Mouser ordercode (none) -> 534-5014
Other:
- note added: "DNP"
